File: CAD/V1.2.2/EasyC_LCD_Driver.kicad_pcb (KiCad board)
At the start: 2 copper layers, 54 x 22 mm, 71 parts, among them K1 easyC-SMD, K2 easyC-SMD, K3 HEADER_MALE_8X1, K4 HEADER_MALE_8X1, K5 HEADER_MALE_4X1, Q1 NMOS-SOT-23-3, U1 TCA9534PWR, U2 TPS613222A, U3 NMOS-DUAL

Commit message: Updating open source files.
Parts:
- C3: value 1uF -> 1u
- C4: value 0.1uF -> 100n
- Q1: value NMOS-SOT-23-3 -> NMOS
- renumbered JP4 to JP1, JP5 to JP2, JP1 to JP3, JP2 to JP4, JP3 to JP5
Changed lines of the file:
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@@
     (title "easyC LCD driver")
     (date "2021-06-09")
-    (rev "V1.1.1.")
+    (rev "V1.2.2.")
     (company "SOLDERED")
     (comment 1 "333003")
@@
       (effects (font (size 1 1) (thickness 0.15)))
     )
-    (fp_text value "0.1uF" (at 0 1.5 180 unlocked) (layer "F.Fab")
+    (fp_text value "100n" (at 0 1.5 180 unlocked) (layer "F.Fab")
       (effects (font (size 1 1) (thickness 0.15)))
     )
@@
     (property "Sheetfile" "EasyC_LCD_Driver.kicad_sch")
     (property "Sheetname" "")
-    (fp_text reference "JP2" (at -0.04 -1.24 90 unlocked) (layer "User.1")
+    (fp_text reference "JP4" (at -0.04 -1.24 90 unlocked) (layer "User.1")
       (effects (font (size 1 1) (thickness 0.15)))
     )
@@
       (effects (font (size 1 1) (thickness 0.15)))
     )
-    (fp_text value "NMOS-SOT-23-3" (at 0 2.7 unlocked) (layer "F.Fab")
+    (fp_text value "NMOS" (at 0 2.7 unlocked) (layer "F.Fab")
       (effects (font (size 1 1) (thickness 0.15)))
     )
@@
     (property "Sheetfile" "EasyC_LCD_Driver.kicad_sch")
     (property "Sheetname" "")
-    (fp_text reference "JP1" (at -0.04 -1.24 90 unlocked) (layer "User.1")
+    (fp_text reference "JP3" (at -0.04 -1.24 90 unlocked) (layer "User.1")
       (effects (font (size 1 1) (thickness 0.15)))
     )
@@
     (property "Sheetfile" "EasyC_LCD_Driver.kicad_sch")
     (property "Sheetname" "")
-    (fp_text reference "JP4" (at 0 -1.5 180 unlocked) (layer "User.1")
+    (fp_text reference "JP1" (at 0 -1.5 180 unlocked) (layer "User.1")
       (effects (font (size 1 1) (thickness 0.15)))
     )
@@
     (property "Sheetfile" "EasyC_LCD_Driver.kicad_sch")
     (property "Sheetname" "")
-    (fp_text reference "JP5" (at 0 -1.5 180 unlocked) (layer "User.1")
+    (fp_text reference "JP2" (at 0 -1.5 180 unlocked) (layer "User.1")
       (effects (font (size 1 1) (thickness 0.15)))
     )
@@
     (property "Sheetfile" "EasyC_LCD_Driver.kicad_sch")
     (property "Sheetname" "")
-    (fp_text reference "JP3" (at -0.04 -1.24 90 unlocked) (layer "User.1")
+    (fp_text reference "JP5" (at -0.04 -1.24 90 unlocked) (layer "User.1")
       (effects (font (size 1 1) (thickness 0.15)))
     )
@@
       (effects (font (size 1 1) (thickness 0.15)))
     )
-    (fp_text value "1uF" (at 0 1.5 180 unlocked) (layer "F.Fab")
+    (fp_text value "1u" (at 0 1.5 180 unlocked) (layer "F.Fab")
       (effects (font (size 1 1) (thickness 0.15)))
     )
