File: CAD/V1.2.2/EasyC_LCD_Driver.kicad_sch (KiCad schematic)
At the start: 33 parts, among them K1 easyC-SMD, K2 easyC-SMD, K3 HEADER_MALE_8X1, K4 HEADER_MALE_8X1, K5 HEADER_MALE_4X1, Q1 NMOS, U1 TCA9534PWR, U2 TPS613222A, U3 NMOS-DUAL

Commit message: Updating open source files.
Parts:
- renumbered JP4 to JP1, JP5 to JP2, JP1 to JP3, JP2 to JP4, JP3 to JP5
Changed lines of the file:
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@@
     (title "easyC LCD driver")
     (date "2021-06-09")
-    (rev "V1.1.1.")
+    (rev "V1.2.2.")
     (company "SOLDERED")
     (comment 1 "333003")
@@
   (symbol (lib_id "e-radionica.com schematics:SMD_JUMPER_3_PAD_TRACE") (at 53.34 125.73 180) (unit 1)
     (in_bom yes) (on_board yes)
-    (property "Reference" "JP4" (id 0) (at 54.61 128.27 0))
+    (property "Reference" "JP1" (id 0) (at 54.61 128.27 0))
     (property "Value" "SMD_JUMPER_3_PAD_TRACE" (id 1) (at 53.34 129.54 0)
       (effects (font (size 1.27 1.27)) hide)
@@
   (symbol (lib_id "e-radionica.com schematics:SMD_JUMPER") (at 130.81 51.435 90) (unit 1)
     (in_bom yes) (on_board yes)
-    (property "Reference" "JP3" (id 0) (at 130.81 51.435 90)
+    (property "Reference" "JP5" (id 0) (at 130.81 51.435 90)
       (effects (font (size 1.27 1.27)) (justify right))
     )
@@
   (symbol (lib_id "e-radionica.com schematics:SMD_JUMPER") (at 110.49 51.435 90) (unit 1)
     (in_bom yes) (on_board yes)
-    (property "Reference" "JP1" (id 0) (at 110.49 51.435 90)
+    (property "Reference" "JP3" (id 0) (at 110.49 51.435 90)
       (effects (font (size 1.27 1.27)) (justify right))
     )
@@
   (symbol (lib_id "e-radionica.com schematics:SMD_JUMPER") (at 120.65 51.435 90) (unit 1)
     (in_bom yes) (on_board yes)
-    (property "Reference" "JP2" (id 0) (at 120.65 51.435 90)
+    (property "Reference" "JP4" (id 0) (at 120.65 51.435 90)
       (effects (font (size 1.27 1.27)) (justify right))
     )
@@
   (symbol (lib_id "e-radionica.com schematics:SMD_JUMPER_3_PAD_TRACE") (at 93.98 125.73 180) (unit 1)
     (in_bom yes) (on_board yes)
-    (property "Reference" "JP5" (id 0) (at 95.25 128.27 0))
+    (property "Reference" "JP2" (id 0) (at 95.25 128.27 0))
     (property "Value" "SMD_JUMPER_3_PAD_TRACE" (id 1) (at 93.98 129.54 0)
       (effects (font (size 1.27 1.27)) hide)
@@
       (reference "H2") (unit 1) (value "HOLE_3.2mm") (footprint "e-radionica.com footprinti:HOLE_3.2mm")
     )
+    (path "/2b49e721-ea38-4a64-8a71-f29377eba848"
+      (reference "JP1") (unit 1) (value "SMD_JUMPER_3_PAD_TRACE") (footprint "e-radionica.com footprinti:SMD_JUMPER_3_PAD_TRACE")
+    )
+    (path "/ee854cff-3cfa-4451-8c61-0b4083d5bd90"
+      (reference "JP2") (unit 1) (value "SMD_JUMPER_3_PAD_TRACE") (footprint "e-radionica.com footprinti:SMD_JUMPER_3_PAD_TRACE")
+    )
     (path "/b8e36e78-68ff-435c-bf6e-b1d0c7d5ec82"
-      (reference "JP1") (unit 1) (value "SMD_JUMPER") (footprint "e-radionica.com footprinti:SMD_JUMPER")
+      (reference "JP3") (unit 1) (value "SMD_JUMPER") (footprint "e-radionica.com footprinti:SMD_JUMPER")
     )
     (path "/dc076157-bc0f-4f8c-9ad5-ee40dc09fe70"
-      (reference "JP2") (unit 1) (value "SMD_JUMPER") (footprint "e-radionica.com footprinti:SMD_JUMPER")
+      (reference "JP4") (unit 1) (value "SMD_JUMPER") (footprint "e-radionica.com footprinti:SMD_JUMPER")
     )
     (path "/8d8e243d-b0f0-425e-9459-263c8975d766"
-      (reference "JP3") (unit 1) (value "SMD_JUMPER") (footprint "e-radionica.com footprinti:SMD_JUMPER")
-    )
-    (path "/2b49e721-ea38-4a64-8a71-f29377eba848"
-      (reference "JP4") (unit 1) (value "SMD_JUMPER_3_PAD_TRACE") (footprint "e-radionica.com footprinti:SMD_JUMPER_3_PAD_TRACE")
-    )
-    (path "/ee854cff-3cfa-4451-8c61-0b4083d5bd90"
-      (reference "JP5") (unit 1) (value "SMD_JUMPER_3_PAD_TRACE") (footprint "e-radionica.com footprinti:SMD_JUMPER_3_PAD_TRACE")
+      (reference "JP5") (unit 1) (value "SMD_JUMPER") (footprint "e-radionica.com footprinti:SMD_JUMPER")
     )
     (path "/fcd02546-df7a-4ae6-8c7e-ba267fa354ba"

Commit message: Updating open source files.
Other:
- note removed: "Stavljeni su 0805 footprinti za sva 3 kondenzatora jer su 0603 footprinti mali za te kondenzatore koji su veći od generic 0603C"
- note removed: "ZAMJENA za CL10A226MPCNUBE treba probati CL10A226MP8NUNE"
Changed lines of the file:
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@@
   (junction (at 120.65 57.785) (diameter 0.9144) (color 0 0 0 0)
   )
+  (junction (at 195.58 124.46) (diameter 0) (color 0 0 0 0)
+  )
   (junction (at 63.5 104.14) (diameter 0.9144) (color 0 0 0 0)
   )
@@
   (junction (at 107.95 163.83) (diameter 0.9144) (color 0 0 0 0)
   )
-  (junction (at 195.58 124.206) (diameter 0.9144) (color 0 0 0 0)
-  )
   (junction (at 130.81 57.785) (diameter 0.9144) (color 0 0 0 0)
   )
@@
   )
   (wire (pts (xy 63.5 99.06) (xy 63.5 104.14))
-    (stroke (width 0) (type solid) (color 0 0 0 0))
-  )
-  (wire (pts (xy 198.12 124.206) (xy 195.58 124.206))
     (stroke (width 0) (type solid) (color 0 0 0 0))
   )
@@
     (stroke (width 0) (type solid) (color 0 0 0 0))
   )
+  (wire (pts (xy 198.12 124.46) (xy 195.58 124.46))
+    (stroke (width 0) (type default) (color 0 0 0 0))
+  )
   (wire (pts (xy 55.88 161.925) (xy 55.88 160.02))
     (stroke (width 0) (type solid) (color 0 0 0 0))
@@
     (stroke (width 0) (type solid) (color 0 0 0 0))
   )
+  (wire (pts (xy 189.23 124.46) (xy 195.58 124.46))
+    (stroke (width 0) (type default) (color 0 0 0 0))
+  )
   (wire (pts (xy 43.18 62.23) (xy 45.72 62.23))
     (stroke (width 0) (type solid) (color 0 0 0 0))
@@
     (stroke (width 0) (type solid) (color 0 0 0 0))
   )
-  (wire (pts (xy 193.04 124.46) (xy 195.58 124.46))
-    (stroke (width 0) (type solid) (color 0 0 0 0))
-  )
-  (wire (pts (xy 195.58 121.285) (xy 195.58 124.206))
-    (stroke (width 0) (type solid) (color 0 0 0 0))
-  )
-  (wire (pts (xy 195.58 124.206) (xy 195.58 124.46))
+  (wire (pts (xy 195.58 121.285) (xy 195.58 124.46))
     (stroke (width 0) (type solid) (color 0 0 0 0))
   )
@@
     (stroke (width 0) (type solid) (color 0 0 0 0))
   )
-  (text "Stavljeni su 0805 footprinti za sva 3 kondenzatora\njer su 0603 footprinti mali za te kondenzatore\nkoji su veći od generic 0603C\n"
-    (at 68.58 185.42 0)
-    (effects (font (size 1.27 1.27)) (justify right bottom))
-  )
   (text "I2C ADDRESS SELECTION" (at 130.81 30.48 180)
     (effects (font (size 1.27 1.27)) (justify right bottom))
@@
     (effects (font (size 1.27 1.27)) (justify right bottom))
   )
-  (text "ZAMJENA za CL10A226MPCNUBE treba probati\nCL10A226MP8NUNE"
-    (at 57.15 157.48 0)
-    (effects (font (size 1.27 1.27)) (justify right bottom))
-  )
   (text "BOOST CONVERTER 3V3>>5V" (at 54.61 148.59 180)
     (effects (font (size 1.27 1.27)) (justify right bottom))
@@
     )
   )
-  (global_label "P3" (shape input) (at 193.04 124.46 180)
-    (effects (font (size 1.27 1.27)) (justify right))
-    (property "Intersheet References" "${INTERSHEET_REFS}" (id 0) (at 186.6234 124.3806 0)
+  (global_label "P3" (shape input) (at 189.23 124.46 180)
+    (effects (font (size 1.27 1.27)) (justify right))
+    (property "Intersheet References" "${INTERSHEET_REFS}" (id 0) (at 182.8134 124.3806 0)
       (effects (font (size 1.27 1.27)) (justify right) hide)
     )
@@
     (pin "3")
   )
-  (symbol (lib_id "e-radionica.com schematics:3V3") (at 191.135 52.07 0) (unit 1)
+  (symbol (lib_name "3V3_1") (lib_id "e-radionica.com schematics:3V3") (at 191.135 52.07 0) (unit 1)
     (in_bom yes) (on_board yes)
     (property "Reference" "#PWR012" (id 0) (at 195.58 52.07 0)
@@
     )
   )
-  (symbol (lib_id "e-radionica.com schematics:5V") (at 250.19 57.15 0) (unit 1)
+  (symbol (lib_name "5V_4") (lib_id "e-radionica.com schematics:5V") (at 250.19 57.15 0) (unit 1)
     (in_bom yes) (on_board yes)
     (property "Reference" "#PWR025" (id 0) (at 254.635 57.15 0)
@@
     (pin "1")
   )
-  (symbol (lib_id "e-radionica.com schematics:5V") (at 59.69 156.21 0) (unit 1)
+  (symbol (lib_name "5V_6") (lib_id "e-radionica.com schematics:5V") (at 59.69 156.21 0) (unit 1)
     (in_bom yes) (on_board yes)
     (property "Reference" "#PWR03" (id 0) (at 64.135 156.21 0)
@@
     (pin "2")
   )
-  (symbol (lib_id "e-radionica.com schematics:GND") (at 55.88 172.72 0) (unit 1)
+  (symbol (lib_name "GND_8") (lib_id "e-radionica.com schematics:GND") (at 55.88 172.72 0) (unit 1)
     (in_bom yes) (on_board yes)
     (property "Reference" "#PWR02" (id 0) (at 60.325 172.72 0)
@@
     (pin "1")
   )
-  (symbol (lib_id "e-radionica.com schematics:GND") (at 231.14 146.05 0) (unit 1)
+  (symbol (lib_name "GND_6") (lib_id "e-radionica.com schematics:GND") (at 231.14 146.05 0) (unit 1)
     (in_bom yes) (on_board yes)
     (property "Reference" "#PWR021" (id 0) (at 235.585 146.05 0)
@@
     (pin "9")
   )
-  (symbol (lib_id "e-radionica.com schematics:GND") (at 82.55 170.18 0) (unit 1)
+  (symbol (lib_name "GND_9") (lib_id "e-radionica.com schematics:GND") (at 82.55 170.18 0) (unit 1)
     (in_bom yes) (on_board yes)
     (property "Reference" "#PWR07" (id 0) (at 86.995 170.18 0)
@@
     (pin "2")
   )
-  (symbol (lib_id "e-radionica.com schematics:3V3") (at 211.455 52.07 0) (unit 1)
+  (symbol (lib_name "3V3_2") (lib_id "e-radionica.com schematics:3V3") (at 211.455 52.07 0) (unit 1)
     (in_bom yes) (on_board yes)
     (property "Reference" "#PWR016" (id 0) (at 215.9 52.07 0)
@@
     (pin "1")
   )
-  (symbol (lib_id "e-radionica.com schematics:5V") (at 53.34 121.92 0) (unit 1)
+  (symbol (lib_name "5V_7") (lib_id "e-radionica.com schematics:5V") (at 53.34 121.92 0) (unit 1)
     (in_bom yes) (on_board yes)
     (property "Reference" "#PWR04" (id 0) (at 57.785 121.92 0)
@@
     (pin "2")
   )
-  (symbol (lib_id "e-radionica.com schematics:3V3") (at 82.55 106.68 270) (unit 1)
+  (symbol (lib_name "3V3_3") (lib_id "e-radionica.com schematics:3V3") (at 82.55 106.68 270) (unit 1)
     (in_bom yes) (on_board yes)
     (property "Reference" "#PWR022" (id 0) (at 82.55 111.125 0)
@@
     (pin "1")
   )
-  (symbol (lib_id "e-radionica.com schematics:GND") (at 107.95 173.99 0) (unit 1)
+  (symbol (lib_name "GND_10") (lib_id "e-radionica.com schematics:GND") (at 107.95 173.99 0) (unit 1)
     (in_bom yes) (on_board yes)
     (property "Reference" "#PWR09" (id 0) (at 112.395 173.99 0)
@@
     (pin "1")
   )
-  (symbol (lib_id "e-radionica.com schematics:3V3") (at 64.77 106.68 90) (unit 1)
+  (symbol (lib_name "3V3_5") (lib_id "e-radionica.com schematics:3V3") (at 64.77 106.68 90) (unit 1)
     (in_bom yes) (on_board yes)
     (property "Reference" "#PWR020" (id 0) (at 64.77 102.235 0)
@@
     (pin "2")
   )
-  (symbol (lib_id "e-radionica.com schematics:3V3") (at 93.98 121.92 0) (unit 1)
+  (symbol (lib_name "3V3_4") (lib_id "e-radionica.com schematics:3V3") (at 93.98 121.92 0) (unit 1)
     (in_bom yes) (on_board yes)
     (property "Reference" "#PWR023" (id 0) (at 98.425 121.92 0)
@@
     (pin "1")
   )
-  (symbol (lib_id "e-radionica.com schematics:5V") (at 217.17 104.14 0) (unit 1)
+  (symbol (lib_name "5V_3") (lib_id "e-radionica.com schematics:5V") (at 217.17 104.14 0) (unit 1)
     (in_bom yes) (on_board yes)
     (property "Reference" "#PWR018" (id 0) (at 221.615 104.14 0)
@@
     (pin "8")
   )
-  (symbol (lib_id "e-radionica.com schematics:GND") (at 76.2 46.99 0) (unit 1)
+  (symbol (lib_name "GND_7") (lib_id "e-radionica.com schematics:GND") (at 76.2 46.99 0) (unit 1)
     (in_bom yes) (on_board yes)
     (property "Reference" "#PWR06" (id 0) (at 80.645 46.99 0)
@@
     (pin "1")
   )
-  (symbol (lib_id "e-radionica.com schematics:5V") (at 195.58 111.76 0) (unit 1)
+  (symbol (lib_name "5V_2") (lib_id "e-radionica.com schematics:5V") (at 195.58 111.76 0) (unit 1)
     (in_bom yes) (on_board yes)
     (property "Reference" "#PWR014" (id 0) (at 200.025 111.76 0)
@@
     (pin "2")
   )
-  (symbol (lib_id "e-radionica.com schematics:GND") (at 246.38 62.23 0) (unit 1)
+  (symbol (lib_name "GND_4") (lib_id "e-radionica.com schematics:GND") (at 246.38 62.23 0) (unit 1)
     (in_bom yes) (on_board yes)
     (property "Reference" "#PWR024" (id 0) (at 250.825 62.23 0)
       (effects (font (size 1 1)) hide)
     )
-    (property "Value" "GND" (id 1) (at 246.38 64.77 0)
+    (property "Value" "GND" (id 1) (at 246.38 65.405 0)
       (effects (font (size 1 1)))
     )
@@
     (pin "1")
   )
-  (symbol (lib_id "e-radionica.com schematics:5V") (at 218.44 139.7 90) (unit 1)
+  (symbol (lib_name "5V_5") (lib_id "e-radionica.com schematics:5V") (at 218.44 139.7 90) (unit 1)
     (in_bom yes) (on_board yes)
     (property "Reference" "#PWR019" (id 0) (at 218.44 135.255 0)
@@
     (pin "1")
   )
-  (symbol (lib_id "e-radionica.com schematics:GND") (at 200.66 129.54 0) (unit 1)
+  (symbol (lib_name "GND_5") (lib_id "e-radionica.com schematics:GND") (at 200.66 129.54 0) (unit 1)
     (in_bom yes) (on_board yes)
     (property "Reference" "#PWR015" (id 0) (at 205.105 129.54 0)
       (effects (font (size 1 1)) hide)
     )
-    (property "Value" "GND" (id 1) (at 200.66 133.35 0)
+    (property "Value" "GND" (id 1) (at 200.66 132.715 0)
       (effects (font (size 1 1)))
     )
@@
     (pin "1")
   )
-  (symbol (lib_id "e-radionica.com schematics:GND") (at 211.455 64.77 0) (unit 1)
+  (symbol (lib_name "GND_2") (lib_id "e-radionica.com schematics:GND") (at 211.455 64.77 0) (unit 1)
     (in_bom yes) (on_board yes)
     (property "Reference" "#PWR017" (id 0) (at 215.9 64.77 0)
       (effects (font (size 1 1)) hide)
     )
-    (property "Value" "GND" (id 1) (at 211.455 68.58 0)
+    (property "Value" "GND" (id 1) (at 211.455 67.945 0)
       (effects (font (size 1 1)))
     )
@@
     (pin "2")
   )
-  (symbol (lib_id "e-radionica.com schematics:GND") (at 191.135 64.77 0) (unit 1)
+  (symbol (lib_name "GND_3") (lib_id "e-radionica.com schematics:GND") (at 191.135 64.77 0) (unit 1)
     (in_bom yes) (on_board yes)
     (property "Reference" "#PWR013" (id 0) (at 195.58 64.77 0)
       (effects (font (size 1 1)) hide)
     )
-    (property "Value" "GND" (id 1) (at 191.135 68.58 0)
-      (effects (font (size 1 1)))
-    )
+    (property "Value" "GND" (id 1) (at 191.135 67.945 0)
+      (effects (font (size 1 1)))
+    )
